File: pocket_radio_v3.kicad_sch (KiCad schematic)
At the start: 19 parts, among them J1 54-00174, SW1 SW_Push, SW2 SW_Push, U1 STM32G030C8Tx, U2 Si4704/05-D60-GM, U3 TPA6111A2D, U4 MAX809STRG, U5 LDL1117S50R, U6 LDL1117S33R, Y1 Crystal, Y2 Crystal

Commit message: Amost done schematic
Parts:
- added AE1: Antenna, symbol Device:Antenna
- added C10, C9: 22pF, symbol Device:C
- added C11, C12, C13, C14, C15, C18, C23: 0.1uF, symbol Device:C
- added C16, C8: 7.5pF, symbol Device:C
- added C17: 22nF, symbol Device:C
- added C19, C20: 0.39uF, symbol Device:C
- added C21, C22: 5pF, symbol Device:C
- added C24: 1uF, symbol Device:C
- added C25, C26: 68uF, symbol Device:C
- added D1, D2, D3, D4, D5: LED, symbol Device:LED
- added J2: Conn_01x07_Pin, symbol Connector:Conn_01x07_Pin
- added J3: Conn_01x04_Pin, symbol Connector:Conn_01x04_Pin
- added L1: 120nH, symbol Device:L
- added R1, R2, R3, R4, R5: 200R, symbol Device:R_US
- added R10, R11: 4.7k, symbol Device:R_US
- added R12, R13: 2k, symbol Device:R_US
- added R14, R16: 20k, symbol Device:R_US
- added R15, R17: 200k, symbol Device:R_US
- added R6, R7, R8, R9: 10k, symbol Device:R_US
- added SW3, SW4, SW5: SW_Push, Button_Switch_SMD:SW_SPST_PTS647_Sx38, symbol Switch:SW_Push
- added TP1, TP2, TP3, TP4: TestPoint, symbol Connector:TestPoint
- U2: value Si4704/05-D60-GM -> Si4704-D60-GM
- Y1: value Crystal -> 8MHz
Connections:
- net +3.3V: now also U2.10 (VD), U4.3 (VCC), C18.1, J2.1 (Pin_1), R10.2, R11.2; no longer U1.5 (VREF+)
- net +5VA: now also U2.11 (VA), U3.8 (VDD), C17.2, C23.1
- net GND: now also J1.1 (MIC), J1.2 (GND), SW1.2, U2.12 (GND), U2.15 (DOUT), U2.16 (DFS), U2.2 (FMI), U2.3 (RFGND), U2.EP (21), U3.4 (GND), U3.5 (SHDN), U4.1 (GND), C10.1, C11.2, C12.1, C12.2, C13.1, C13.2, C14.1, C14.2, C15.1, C15.2, C16.1, C17.1, C18.2, C23.2, C24.2, C8.1, C9.1, J2.3 (Pin_3), J2.5 (Pin_5), J2.6 (Pin_6), L1.2, R1.1, R2.1, R3.1, R4.1, R5.1, SW3.2, SW4.2, SW5.2
- net NRST: now reaches C7.1, SW2.2, U1.10 (NRST)
- net NRST: now also J2.7 (Pin_7)
- net at Y2.1: now also U2.17 (GPO3), C16.2
- net at Y2.2: now also U2.9 (RCLK), C8.2
- net at U1.11 (PA0): now also J3.1 (Pin_1)
- net at U1.12 (PA1): now also J3.2 (Pin_2)
- net at U1.13 (PA2): now also J3.3 (Pin_3)
- net at U1.14 (PA3): now also J3.4 (Pin_4)
- net at U1.19 (PB0): now also R6.2
- net at U1.20 (PB1): now also R7.2
- net at U1.21 (PB2): now also R8.2
- net ADDR_SEL: now reaches U1.22 (PB10)
- net ADDR_SEL: now also U2.6 (~{SEN})
- net at U1.23 (PB11): now also D1.2 (A)
- net at U1.24 (PB12): now also D2.2 (A)
- net at U1.25 (PB13): now also D3.2 (A)
- net at U1.26 (PB14): now also D4.2 (A)
- net at U1.27 (PB15): now also D5.2 (A)
- net at U1.35 (PA13): now also J2.2 (Pin_2)
- net at U1.36 (PA14): now also J2.4 (Pin_4)
- net at U1.42 (PB3): now also R9.2
- net at U1.45 (PB6): now also R12.2
- net at U1.46 (PB7): now also R13.2
- net GPO1: now reaches U1.47 (PB8)
- net GPO1: now also U2.19 (GPO1)
- net GPO2: now reaches U1.48 (PB9)
- net GPO2: now also U2.18 (GPO2)
- net at U1.8 (PF0): now also Y1.2, C9.2
- net at U1.9 (PF1): now also Y1.1, C10.2
- net at U3.1 (VO1): now also C25.2
- net at U3.2 (IN1-): now also R14.1, R15.2
- net at U3.3 (BYPASS): now also C24.1
- net at U3.6 (IN2-): now also R16.1, R17.2
- net at U3.7 (VO2): now also C26.2
- net at U2.13 (ROUT): now also C19.2, TP1.1
- net at U2.14 (LOUT): now also C20.2, TP2.1
- net at U2.4 (LPI): now also AE1.1 (A), L1.1
- net at U2.5 (~{RST}): now also U4. (~{RST})
- net SCL: now reaches U2.7 (SCLK)
- net SCL: now also R10.1, R12.1, TP3.1
- net SDA: now reaches U2.8 (SDIO)
- net SDA: now also R11.1, R13.1, TP4.1
- net at SW1.1: now also R6.1
- net at J1.3 (R): now also C25.1
- net at J1.4 (L): now also C26.1
- new net: D3.1 (K), R3.2
- new net: D4.1 (K), R4.2
- new net: C11.1, U1.5 (VREF+)
- new net: R8.1, SW4.1
- new net: C19.1, R14.2
- new net: R9.1, SW5.1
- new net: C21.2, R15.1
- new net: D2.1 (K), R2.2
- new net: C22.2, R17.1
- new net: C20.1, R16.2
- new net: D5.1 (K), R5.2
- new net: R7.1, SW3.1
- new net: D1.1 (K), R1.2
- no-connect marks 0 -> 19
Other:
- note added: "ADCs and DACs not used, so VREF can be grounded"
- note added: "Audio frequency range: 20Hz-20kHz"
- note added: "C_{L}-C_{S} = 12.5-9 = C^{2}/2C So, C = 7pF"
- note added: "C_{L}-C_{S} = 20-9 = C^{2}/2C So, C = 22pF"
- note added: "Cutoff frequency 73Hz at 32R load"
- note added: "Cutoff frequency = 1 / (2*pi*1MOhm*0.39uF) = 0.41 Hz"
- note added: "Gain = 10. Effective impedance 18.2k is within range 5-20k."
- note added: "L = 1 / ((2*pi*98MHz)^2 * C) Assuming C = 22pF, L = 120nH"
- note added: "Metal film preferred for gain resistors. Low leakage tantalum or ceramic caps for input. Low ESR caps recommended in general."
- note added: "PCB trace embedded antenna"
- note added: "Route unused pins to GND"
- moved on the sheet: C1, C2, C3, C4, C5, C6, C7, FB1, J1, SW1, SW2, U1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

Commit message: Schematic mostly done
Parts:
- removed U1: STM32G030C8Tx, Package_QFP:LQFP-48_7x7mm_P0.5mm, symbol MCU_ST_STM32G0:STM32G030C8Tx
- added C27: 1uF, Capacitor_SMD:C_0603_1608Metric, symbol Device:C
- added H1, H2, H3, H4: MountingHole, symbol Mechanical:MountingHole
- added JP1: Jumper_2_Open, symbol Jumper:Jumper_2_Open
- added R18: 2R, Resistor_SMD:R_0603_1608Metric, symbol Device:R_US
- added U7: STM32G030C8Tx, Package_QFP:LQFP-48_7x7mm_P0.5mm, symbol MCU_ST_STM32G0:STM32G030C8Tx
- AE1, J2, J3: now left out of the parts list
- C1, C24, C3: footprint (none) -> Capacitor_SMD:C_0603_1608Metric; Link (none) -> https://www.digikey.ca/en/products/detail/samsung-electro-m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
- C10, C11, C12, C13, C14, C15, C18, C23, C6, C7, C9: footprint (none) -> Capacitor_SMD:C_0402_1005Metric; Link (none) -> https://www.digikey.ca/en/products/detail/samsung-electro-m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
- C16, C17, C8: footprint (none) -> Capacitor_SMD:C_0402_1005Metric; Link (none) -> https://www.digikey.ca/en/products/detail/murata-electronic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
- C19, C20: footprint (none) -> Capacitor_SMD:C_0603_1608Metric; Link (none) -> https://www.digikey.ca/en/products/detail/yageo/CC0603JRX7R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
- C2, C4, C5: footprint (none) -> Capacitor_SMD:C_0603_1608Metric; Link (none) -> https://www.digikey.ca/en/products/detail/murata-electronic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
- C21, C22: footprint (none) -> Capacitor_SMD:C_0603_1608Metric; Link (none) -> https://www.digikey.ca/en/products/detail/yageo/CC0603CRNPO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
- C25, C26: footprint (none) -> Capacitor_SMD:C_1210_3225Metric; Link (none) -> https://www.digikey.ca/en/products/detail/murata-electronic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
- D1, D2, D3, D4, D5: footprint (none) -> Diode_SMD:D_0603_1608Metric; Link (none) -> https://www.digikey.ca/en/products/detail/liteon/LTST-C190G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
- FB1: Link (none) -> https://www.digikey.ca/en/products/detail/tdk-corporation/M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
- J1: Link (none) -> https://www.digikey.ca/en/products/detail/tensility-interna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
- L1: footprint (none) -> Inductor_SMD:L_0603_1608Metric; Link (none) -> https://www.digikey.ca/en/products/detail/murata-electronic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
- R1, R2, R3, R4, R5: value 200R -> 470R; footprint (none) -> Resistor_SMD:R_0603_1608Metric; Link (none) -> https://www.digikey.ca/en/products/detail/te-connectivity-p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
- R10, R11: footprint (none) -> Resistor_SMD:R_0603_1608Metric; Link (none) -> https://www.digikey.ca/en/products/detail/yageo/RC0603FR-07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
- R12, R13: footprint (none) -> Resistor_SMD:R_0603_1608Metric; Link (none) -> https://www.digikey.ca/en/products/detail/panasonic-electro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
- R14, R16: footprint (none) -> Resistor_SMD:R_0603_1608Metric; Link (none) -> https://www.digikey.ca/en/products/detail/koa-speer-electro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
- R15, R17: footprint (none) -> Resistor_SMD:R_0805_2012Metric; Link (none) -> https://www.digikey.ca/en/products/detail/koa-speer-electro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
- R6, R7, R8, R9: footprint (none) -> Resistor_SMD:R_0603_1608Metric; Link (none) -> https://www.digikey.ca/en/products/detail/stackpole-electro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
- SW1, SW2, SW3, SW4, SW5: Link (none) -> https://www.digikey.ca/en/products/detail/c-k/PTS647SK38SMT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
- TP1, TP2, TP3, TP4: footprint (none) -> TestPoint:TestPoint_Pad_D1.5mm; now left out of the parts list
Connections:
- net +3.3V: now also U7.4 (VBAT), U7.6 (VDD)
- net +5VA: now also C27.1
- net ADDR_SEL: now also U7.22 (PB10)
- net GND: now also JP1.2 (B), R18.1, U7.7 (VSS)
- net GPO1: now also U7.47 (PB8)
- net GPO2: now also U7.48 (PB9)
- net NRST: now also U7.10 (NRST)
- net at C10.2, Y1.1: now also U7.9 (PF1)
- net at R6.2: now also U7.19 (PB0)
- net at C11.1: now also U7.5 (VREF+)
- net at R8.2: now also U7.21 (PB2)
- net at J3.1 (Pin_1): now also U7.11 (PA0)
- net at J3.2 (Pin_2): now also U7.12 (PA1)
- net at J3.3 (Pin_3): now also U7.13 (PA2)
- net at J3.4 (Pin_4): now also U7.14 (PA3)
- net at R7.2: now also U7.20 (PB1)
- net at D1.2 (A): now also U7.23 (PB11)
- net at D2.2 (A): now also U7.24 (PB12)
- net at D3.2 (A): now also U7.25 (PB13)
- net at D4.2 (A): now also U7.26 (PB14)
- net at D5.2 (A): now also U7.27 (PB15)
- net at J2.2 (Pin_2): now also U7.35 (PA13)
- net at J2.4 (Pin_4): now also U7.36 (PA14)
- net at R9.2: now also U7.42 (PB3)
- net at R12.2: now also U7.45 (PB6)
- net at R13.2: now also U7.46 (PB7)
- net at C9.2, Y1.2: now also U7.8 (PF0)
- net at C25.2, U3.1 (VO1): now also C21.1
- net at C26.2, U3.7 (VO2): now also C22.1
- net at U2.5 (~{RST}), U4. (~{RST}): now also JP1.1 (A)
- new net: C27.2, R18.2
Other:
- note added: "CONTROLLER AND USER INTERFACE"
- note added: "Cutoff frequency = 1 / (2*pi*1MOhm*0.39uF) = 0.41 Hz NOTE: Since changed to 0.47uF"
- note added: "Damping required, resonant frequency less than ferrite crossover frequency"
- note added: "FM RECEIVER AND AMPLIFIER"
- note added: "FM frequency 88-108MHz"
- note added: "M3 mounting holes"
- note added: "MOUNTING HOLES"
- note added: "POWER"
- note removed: "Cutoff frequency = 1 / (2*pi*1MOhm*0.39uF) = 0.41 Hz"
- moved on the sheet: C1, C2, C25, C26, C3, C4, FB1, U4, U5, U6

Commit message: Start layout, add sim files
Parts:
- removed C13, C14, C15: 0.1uF, Capacitor_SMD:C_0402_1005Metric, symbol Device:C
- removed R6, R7, R8, R9: 10k, Resistor_SMD:R_0603_1608Metric, symbol Device:R_US
- added C22, C24, C25: 0.1uF, Capacitor_SMD:C_0402_1005Metric, symbol Device:C
- added J4: ExposedPad2, _Project_Library:ExposedPad_2Conn_2x3mm_P3mm, symbol Connector:Conn_01x02_Pin
- AE1: footprint (none) -> _Project_Library:EmbeddedAntenna_Si47xx
- H1, H4: footprint (none) -> MountingHole:MountingHole_3.2mm_M3_ISO7380
- H2: renamed from H3; footprint (none) -> MountingHole:MountingHole_3.2mm_M3_ISO7380
- H3: renamed from H2; footprint (none) -> MountingHole:MountingHole_3.2mm_M3_ISO7380
- J1: renamed from J3; footprint (none) -> _Project_Library:PinHeader_1x04_P2.54mm_Vertical_Tight
- J2: footprint (none) -> _Project_Library:PinHeader_1x07_P2.54mm_Vertical_Tight
- JP1: footprint (none) -> _Project_Library:ViaJumper_Pitch2.54mm_Drill0.7mm
- U1: renamed from U5; Link (none) -> https://www.digikey.ca/en/products/detail/stmicroelectronic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
- U2: renamed from U6; Link (none) -> https://www.digikey.ca/en/products/detail/stmicroelectronic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
- U3: renamed from U4; Link (none) -> https://www.digikey.ca/en/products/detail/onsemi/MAX809STRG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
- U4: renamed from U3; Link (none) -> https://www.digikey.ca/en/products/detail/texas-instruments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
- U5: renamed from U2; Link (none) -> https://www.digikey.ca/en/products/detail/skyworks-solution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
- U6: renamed from U7; Link (none) -> https://www.digikey.ca/en/products/detail/stmicroelectronic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
- Y1: footprint (none) -> _Project_Library:Crystal_SMD_2Pin_11.7x5mm; Link (none) -> https://www.digikey.ca/en/products/detail/fox-electronics/F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
- Y2: value Crystal -> 32.768kHz; footprint (none) -> Crystal:Crystal_SMD_3215-2Pin_3.2x1.5mm; Link (none) -> https://www.digikey.ca/en/products/detail/ecs-inc/ECS-327-1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
- renumbered C27 to C1, C11 to C10, C17 to C11, C18 to C12, C23 to C13, C19 to C14, C20 to C15, C25 to C16, C9 to C17, C26 to C18, C12 to C19, C1 to C2, C24 to C20, C10 to C21, C22 to C23, C8 to C26, C16 to C27, C2 to C3, C3 to C4, C4 to C5, C5 to C7, C7 to C8, C21 to C9, J1 to J3, R18 to R1, R12 to R11, R13 to R12, R1 to R14, R2 to R15, R3 to R16, R4 to R17, R5 to R18, R15 to R2, R14 to R3, R16 to R4, R10 to R6, R11 to R7, R17 to R9, SW2 to SW1, SW1 to SW2
Connections:
- net +9V: now also J4.1 (Pin_1)
- net ADDR_SEL: now also U6.44 (PB5); no longer U6.22 (PB10)
- net GND: now also U5.21 (EP), C22.2, C24.2, C25.2, J4.2 (Pin_2); no longer C19.1, U5.EP (21)
- net at JP1.1 (A), U5.5 (~{RST}): now also U3.2 (~{RST}); no longer U3. (~{RST})
- net at SW2.1: now also C19.1, U6.19 (PB0)
- net at SW4.1: now also U6.21 (PB2), C24.1
- net at R2.2, U4.2 (IN1-): now also C9.2, R4.1; no longer R3.1
- net at C16.2, C9.1, U4.1 (VO1): now also R2.1
- net at R9.2, U4.6 (IN2-): now also C23.2, R3.1; no longer R4.1
- net at C18.2, C23.1, U4.7 (VO2): now also R9.1
- net at SW5.1: now also U6.42 (PB3), C25.1
- net at U6.20 (PB1): now also SW3.1, C22.1
- net at C18.1: now also J3.3 (R); no longer J3.4 (L)
- net at C16.1: now also J3.4 (L); no longer J3.3 (R)
Other:
- moved on the sheet: C1, C10, C17, C19, C2, C21, C23, C3, C4, C5, C6, C7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
