File: pocket_radio_v3.kicad_pcb (KiCad board)
At the start: 4 copper layers, 85 x 55 mm, 76 parts, among them J1 Conn_01x04_Pin, J2 Conn_01x07_Pin, J3 54-00174, J4 ExposedPad2, SW1 SW_Push, SW2 SW_Push, SW3 SW_Push, SW4 SW_Push, SW5 SW_Push, U1 LDL1117S50R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

Commit message: Done layout, except for cosmetics and stitching vias
Parts:
- moved C19 23.2 mm to (98.8, 74.1), turned to -90 degrees
- moved SW2 22.9 mm to (103.0, 74.0), turned to 0 degrees
- moved D1 8.70 mm to (98.5, 52.2), turned to -90 degrees
- moved R14 8.29 mm to (98.5, 48.7), turned to -90 degrees
- moved R18 8.14 mm to (86.5, 48.7), turned to -90 degrees
- moved D5 7.78 mm to (86.5, 52.2), turned to -90 degrees
- moved C25 5.76 mm to (98.8, 81.0)
- moved SW3 5.35 mm to (103.0, 65.0)
- moved D2 4.97 mm to (95.5, 52.2), turned to -90 degrees
- moved R15 4.72 mm to (95.5, 48.7), turned to -90 degrees
- moved R17 4.58 mm to (89.5, 48.7), turned to -90 degrees
- moved D4 4.15 mm to (89.5, 52.2), turned to -90 degrees
- moved TP3 4.01 mm to (71.8, 53.9)
- moved C22 3.97 mm to (98.8, 65.0), turned to -90 degrees
- moved J1 3.94 mm to (90.5, 61.5), turned to 90 degrees
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Routing:
- net +3.3V: track 0.00 -> 123.9 mm, vias 0 -> 12
- net GND: track 0.00 -> 99.6 mm, vias 4 -> 46
- net Net-(U6-PB3): track 0.00 -> 46.1 mm, vias 0 -> 2
- net +5VA: track 0.00 -> 43.4 mm, vias 0 -> 7
- net /SCL: track 0.00 -> 39.5 mm, vias 1 -> 2
- net Net-(U6-PB0): track 0.00 -> 36.8 mm
- net /SDA: track 0.00 -> 36.4 mm, vias 1 -> 2
- net /ADDR_SEL: track 0.00 -> 36.1 mm, vias 1 -> 2
- net /NRST: track 0.00 -> 34.2 mm, vias 0 -> 2
- net /GPO2: track 0.00 -> 32.0 mm
- net /GPO1: track 0.00 -> 31.8 mm
- net Net-(U6-PB1): track 0.00 -> 28.5 mm
- net Net-(U6-PB2): track 0.00 -> 24.5 mm
- net +5V: track 0.00 -> 22.3 mm, vias 1 -> 0
- net Net-(J3-L): track 0.00 -> 21.7 mm
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- added copper zone on B.Cu, net +3.3V
- added copper zone on F.Cu, net +3.3V
- added copper zone on F.Cu, net +5V
- added copper zone on B.Cu, net +5VA
- added copper zone on F.Cu, net +5VA
- added copper zone on F.Cu, net +9V
- added copper zone on In1.Cu, net GND
- added copper zone on In2.Cu, net GND

Commit message: Done and create fab files
Parts:
- moved G*** 72.8 mm to (156.4, 110.8)
- moved C10 69.4 mm to (140.7, 89.5)
- moved C22 69.4 mm to (162.8, 92.0)
- moved AE1 69.4 mm to (109.5, 67.5)
- moved C1 69.4 mm to (123.8, 93.8)
- moved C11 69.4 mm to (108.3, 80.0)
- moved C16 69.4 mm to (116.0, 94.6)
- moved C18 69.4 mm to (107.3, 94.7)
- moved C19 69.4 mm to (162.8, 101.0)
- moved C2 69.4 mm to (121.7, 99.7)
- moved C21 69.4 mm to (147.6, 90.0)
- moved C24 69.4 mm to (162.8, 85.0)
- moved C25 69.4 mm to (162.8, 107.9)
- moved C26 69.4 mm to (108.9, 78.2)
- moved C3 69.4 mm to (126.9, 97.5)
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Routing:
- net GND: track 99.6 -> 106.3 mm, vias 46 -> 90
- net +3.3V: track 123.9 -> 121.7 mm, vias 12 -> 11
- net Net-(D5-K): track 0.00 -> 1.89 mm
- net Net-(D4-K): track 0.00 -> 1.89 mm
- net Net-(D3-K): track 0.00 -> 1.89 mm
- net Net-(D2-K): track 0.00 -> 1.89 mm
- net Net-(D1-K): track 0.00 -> 1.89 mm
- net +5VA: track 43.4 -> 44.0 mm
Other:
- board text added: "+3.3V"
- board text added: "- CHANNEL +"
- board text added: "- VOLUME +"
- board text added: "A.L."
- board text added: "CTS RTS TX RX"
- board text added: "IND 8 4 2 1"
- board text added: "NRST"
- board text added: "POCKET RADIO V3"
- board text added: "POWER (5-9V)"
- board text added: "SWCLK"
- board text added: "SWDIO"
